File: Cheapsk8_LAN.kicad_sch (KiCad schematic)
At the start: 0 parts

Commit message: Changes to be committed: 	modified:   Cheapsk8_LAN.kicad_pcb 	modified:   Cheapsk8_LAN.kicad_prl 	modified:   Cheapsk8_LAN.kicad_pro 	modified:   Cheapsk8_LAN.kicad_sch
 Untracked files:
	Cheapsk8_LAN.csv
	Cheapsk8_LAN.net
	Cheapsk8_LAN.xml
	fp-info-cache
	fp-lib-table
	gerber/
	renders.zip
	sym-lib-table
Parts:
- added C1: 0.1uf, Capacitor_SMD:C_0201_0603Metric_Pad0.64x0.40mm_HandSolder, symbol Device:C
- added C2, C3: 0.1uF, Capacitor_SMD:C_0201_0603Metric_Pad0.64x0.40mm_HandSolder, symbol Device:C
- added C4, C5: 10pF, Capacitor_SMD:C_0201_0603Metric_Pad0.64x0.40mm_HandSolder, symbol Device:C
- added C6, C7: 22uF, Capacitor_THT:CP_Radial_D5.0mm_P2.00mm, symbol Device:C_Polarized_Small_US
- added C8, C9: 0.01uF, Capacitor_SMD:C_0201_0603Metric_Pad0.64x0.40mm_HandSolder, symbol Device:C
- added J2: Bus_ISA_8bit, ISABUS:BUS_PC, symbol Connector:Bus_ISA_8bit
- added J3: SI-50170-F, ISABUS:BEL_SI-50170-F, symbol SI-50170-F:SI-50170-F
- added R14: 27k, Resistor_SMD:R_0603_1608Metric_Pad0.98x0.95mm_HandSolder, symbol Device:R
- added R15: 10k, Resistor_SMD:R_0603_1608Metric_Pad0.98x0.95mm_HandSolder, symbol Device:R
- added R16, R17: 470, Resistor_SMD:R_0603_1608Metric_Pad0.98x0.95mm_HandSolder, symbol Device:R
- added R18: 200, Resistor_SMD:R_0603_1608Metric_Pad0.98x0.95mm_HandSolder, symbol Device:R
- added R19: 1M, Resistor_SMD:R_0603_1608Metric_Pad0.98x0.95mm_HandSolder, symbol Device:R
- added U1: RTL8019AS, ISABUS:RTL8019AS, symbol RTL8019AS:RTL8019AS
- added U2: SST39SF040, Package_DIP:DIP-32_W15.24mm, symbol Memory_Flash:SST39SF040
- added U3: 93LCxxC, Package_DIP:DIP-8_W7.62mm_SMDSocket_SmallPads, symbol Memory_EEPROM:93LCxxC
- added Y1: 20MHz, Crystal:Crystal_HC49-U_Horizontal, symbol Device:Crystal
Connections:
- new net: C4.2, R19.1, U1.51 (X2), Y1.2
- new net: C5.2, R19.2, U1.50 (X1), Y1.1
- new net: C8.1, J3.2 (P2)
- new net: J2.23 (IRQ5), U1.1 (INT3)
- new net: J2.58 (BA04), U1.10 (SA4), U2.8 (A4)
- new net: J2.57 (BA05), U1.11 (SA5), U2.7 (A5)
- new net: J2.56 (BA06), U1.12 (SA6), U2.6 (A6)
- new net: J2.55 (BA07), U1.13 (SA7), U2.5 (A7)
- new net: J2.54 (BA08), U1.15 (SA8), U2.27 (A8)
- new net: J2.53 (BA09), U1.16 (SA9), U2.26 (A9)
- new net: J2.52 (BA10), U1.18 (SA10), U2.23 (A10)
- new net: J2.51 (BA11), U1.19 (SA11), U2.25 (A11)
- new net: J2.24 (IRQ4), U1.2 (INT2)
- new net: J2.50 (BA12), U1.20 (SA12), U2.4 (A12)
- new net: J2.49 (BA13), U1.21 (SA13), U2.28 (A13)
- new net: J2.48 (BA14), U1.22 (SA14)
- new net: J2.47 (BA15), U1.23 (SA15)
- new net: J2.46 (BA16), U1.24 (SA16)
- new net: J2.45 (BA17), U1.25 (SA17)
- new net: J2.44 (BA18), U1.26 (SA18)
- new net: J2.43 (BA19), U1.27 (SA19)
- new net: J2.14 (~{IOR}), U1.29 (IORB)
- new net: J2.25 (IRQ3), U1.3 (INT1)
- new net: J2.13 (~{IOW}), U1.30 (IOWB)
- new net: J2.12 (~{SMEMR}), U1.31 (SMEMRB), U2.24 (OE)
- new net: J2.11 (~{SMEMW}), U1.32 (SMEMWB), U2.31 (PGM)
- new net: J2.2 (RESET), U1.33 (RSTDRV)
- new net: J2.42 (AEN), U1.34 (AEN)
- new net: J2.41 (IO_READY), U1.35 (IOCHRDY)
- new net: J2.40 (DB0), U1.36 (SD0)
- new net: J2.39 (DB1), U1.37 (SD1)
- new net: J2.38 (DB2), U1.38 (SD2)
- new net: J2.37 (DB3), U1.39 (SD3)
- new net: J2.4 (IRQ2), U1.4 (INT0)
- new net: J2.36 (DB4), U1.40 (SD4)
- new net: J2.35 (DB5), U1.41 (SD5)
- new net: J2.34 (DB6), U1.42 (SD6)
- new net: J2.33 (DB7), U1.43 (SD7)
- new net: J3.1 (P1), U1.45 (TPOUT+)
- new net: J3.3 (P3), U1.46 (TPOUT-)
- new net: J2.62 (BA00), U1.5 (SA0), U2.12 (A0)
- new net: J3.6 (P6), R18.2, U1.58 (TPIN-)
- new net: J3.4 (P4), R18.1, U1.59 (TPIN+)
- new net: R17.2, U1.61 (LED0)
- new net: R16.2, U1.62 (LED1)
- new net: R15.2, U1.64 (AUI)
- new net: U1.69 (BA18), U2.1 (A18)
- new net: J2.61 (BA01), U1.7 (SA1), U2.11 (A1)
- new net: U1.71 (BA17), U2.30 (A17)
- new net: U1.72 (BA16), U2.2 (A16)
- new net: U1.73 (BA15), U2.3 (A15)
- new net: U1.74 (BA14), U2.29 (A14)
- new net: U1.75 (BCSB), U2.22 (CE)
- new net: U1.76 (EECS), U3.1 (CS)
- new net: U1.77 (BD7), U2.21 (D7), U3.4 (DO)
- new net: U1.78 (BD6), U2.20 (D6), U3.3 (DI)
- new net: U1.79 (BD5), U2.19 (D5), U3.2 (SCLK)
- new net: J2.60 (BA02), U1.8 (SA2), U2.10 (A2)
- new net: U1.80 (BD4), U2.18 (D4)
- new net: U1.81 (BD3), U2.17 (D3)
- new net: U1.82 (BD2), U2.15 (D2)
- new net: U1.84 (BD1), U2.14 (D1)
- new net: U1.85 (BD0), U2.13 (D0)
- new net: J2.59 (BA03), U1.9 (SA3), U2.9 (A3)
- new net: R14.2, U1.96 (IOCS16B)
- new net: J3.12, R16.1
- new net: J3.10, R17.1
- new net: C9.1, J3.5 (P5)
- new net GND: C1.2, C2.2, C3.2, C4.1, C5.1, C6.2, C7.2, C8.2, C9.2, J2.1 (GND), J2.10 (GND), J2.31 (GND), J3.8 (P8), J3.S1 (SHIELD), J3.S2 (SHIELD), R14.1, R15.1, U1.14 (GND), U1.28 (GND2), U1.44 (GND3), U1.52 (GND4), U1.83 (GND5), U1.86 (GND6), U2.16 (GND), U3.5 (GND)
- new net VCC: C1.1, C2.1, C3.1, C6.1, C7.1, J2.29 (VCC), J2.3 (VCC), J3.11, J3.9, U1.17 (VDD2), U1.47 (VDD3), U1.57 (VDD4), U1.6 (VDD), U1.70 (VDD5), U1.89 (VDD6), U2.32 (VCC), U3.6 (ORG), U3.8 (VCC)
- no-connect marks 0 -> 39
